File: scheme_EAGLE/protractor.sch (EAGLE design)
At the start: 20 parts, among them U1 ATTINY45-20PU

Commit message: Rename the components
Parts:
- R1: value 30k -> 4.7k
- R2: value 1k -> 4.7k
- R6: value 4.7k -> 1k
- R7: value 4.7k -> 30k
- renumbered AC-INPUT to X2, AC-OUTPUT to X1, BT1 to T1
Connections:
- net GND: now also JP2.2; no longer JP1.2
- net N$1: now also D2.A; no longer D1.A
- net N$11: now also JP1.3, R1.1; no longer JP2.3, R7.1
- net N$14: now also JP1.2, JP2.3, R2.1; no longer JP2.2, JP3.3, R6.1
- net N$2: now also D1.C, R7.2; no longer D2.C, R1.2
- net N$4: now also D1.A, D2.C, R6.2; no longer D1.C, D2.A, R2.2
- net N$5: now also R7.1; no longer R1.1
- net N$7: now also R6.1; no longer R2.1
- net VCC: now also JP3.3, R1.2, R2.2; no longer JP1.3, R6.2, R7.2
Other:
- moved on the sheet: D1, D2, JP1, JP2, JP3, R1, R2, R6, R7

Commit message: Now, the firmware is works
Changed lines of the file:
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@@
 <?xml version="1.0" encoding="utf-8"?>
 <!DOCTYPE eagle SYSTEM "eagle.dtd">
-<eagle version="7.2.0">
+<eagle version="7.5.0">
 <drawing>
 <settings>
@@
 <pinref part="JP1" gate="A" pin="2"/>
 <pinref part="R2" gate="G$1" pin="1"/>
-<wire x1="-55.88" y1="60.96" x2="-45.72" y2="60.96" width="0.1524" layer="91"/>
-<wire x1="-45.72" y1="60.96" x2="-43.18" y2="66.04" width="0.1524" layer="91"/>
-<wire x1="-45.72" y1="60.96" x2="-25.4" y2="60.96" width="0.1524" layer="91"/>
-<wire x1="-25.4" y1="60.96" x2="-25.4" y2="66.04" width="0.1524" layer="91"/>
+<wire x1="-55.88" y1="60.96" x2="-48.26" y2="60.96" width="0.1524" layer="91"/>
+<wire x1="-48.26" y1="60.96" x2="-43.18" y2="66.04" width="0.1524" layer="91"/>
+<wire x1="-48.26" y1="60.96" x2="-27.94" y2="60.96" width="0.1524" layer="91"/>
+<wire x1="-27.94" y1="60.96" x2="-25.4" y2="66.04" width="0.1524" layer="91"/>
 <pinref part="U1" gate="A" pin="PB2"/>
 <wire x1="-25.4" y1="66.04" x2="-10.16" y2="66.04" width="0.1524" layer="91"/>
 <pinref part="JP2" gate="A" pin="3"/>
 <wire x1="-55.88" y1="48.26" x2="-45.72" y2="48.26" width="0.1524" layer="91"/>
-<wire x1="-45.72" y1="48.26" x2="-45.72" y2="60.96" width="0.1524" layer="91"/>
-</segment>
-</net>
+<wire x1="-45.72" y1="48.26" x2="-48.26" y2="60.96" width="0.1524" layer="91"/>
+</segment>
+</net>
