File: scheme_EAGLE/protractor2.brd (EAGLE design)
At the start: 52 x 54.3 mm, 20 parts, among them T1 BT136, U1 ATTINY45-20PU

Commit message: Now, the firmware is works
Parts:
- 85: value ATTINY45-20PU -> attiny
- renumbered U1 to 85
Routing:
- net N$9: track 27.6 -> 58.7 mm
- net GND: track 95.9 -> 115.5 mm
- net N$3: track 160.0 -> 179.0 mm
- net N$5: track 55.7 -> 37.4 mm
- net N$14: track 48.7 -> 33.6 mm
- net N$6: track 23.3 -> 31.4 mm
- net N$1: track 39.9 -> 46.3 mm
- net N$12: track 11.2 -> 6.13 mm
- net N$11: track 37.0 -> 33.8 mm
- net N$10: track 16.6 -> 14.8 mm
- net VCC: track 58.8 -> 59.7 mm
- net N$13: track 32.6 -> 33.4 mm
- net N$4: track 82.5 -> 81.8 mm
- net N$8: track 29.1 -> 29.8 mm
- added copper zone on layer 16, net GND
Other:
- board size 52 x 54.3 mm -> 53.3 x 56.2 mm
- board text added: "ATdimmer v1.0"
- board text added: "GND 5V"
- board text added: "SCK SDA"
- board text added: "SWITCH"
